Commit message: Changed joint visual for manipulator arm

File: my_simple_manipulator/ros/config/my_robot.urdf (robot description, URDF)
Before this commit: robot my_simple_manipulator, 5 links, 4 joints
Links:
- added link end_effector; visual sphere radius=0.03
- link link1: geometry visual cylinder length=0.1 radius=0.07; visual cylinder length=1.0 radius=0.05
- link link2: geometry visual cylinder length=0.06 radius=0.04; visual cylinder length=0.6 radius=0.03
Joints:
- added joint joint_ee: type fixed, parent link3, child end_effector, origin xyz=0.4 0.0 0.0 rpy=0 0 0.0, axis 0 0 1

Commit message: Added joint limits to manipulator urdf

File: my_simple_manipulator/ros/config/my_robot.urdf (robot description, URDF)
Before this commit: robot my_simple_manipulator, 6 links, 5 joints
Joints:
- joint joint1: limit (none) -> lower=-3.13 upper=3.13 effort=30 velocity=1.0; type continuous -> revolute
- joint joint2: limit (none) -> lower=-2.13 upper=2.13 effort=30 velocity=1.0; type continuous -> revolute
- joint joint3: limit (none) -> lower=-2.13 upper=2.13 effort=30 velocity=1.0; type continuous -> revolute
