Commit message: Added inertia and controller info for gazebo sim

File: my_simple_manipulator/ros/config/my_robot.xacro (robot description, xacro)
@@ -4,8 +4,42 @@
     <xacro:property name="link2_length" value="0.6" />
     <xacro:property name="link3_length" value="0.4" />
+    <xacro:property name="base_length" value="0.5" />
     <xacro:property name="link1_radius" value="0.05" />
     <xacro:property name="link2_radius" value="0.03" />
     <xacro:property name="link3_radius" value="0.02" />
-    <xacro:property name="base_length" value="0.5" />
+    <xacro:property name="link1_mass" value="1.0" />
+    <xacro:property name="link2_mass" value="0.6" />
+    <xacro:property name="link3_mass" value="0.4" />
+    <xacro:property name="base_mass" value="10.0" />
+    <xacro:property name="ee_mass" value="0.2" />
+    <!-- collision_shortening_factor -->
+    <xacro:property name="csf" value="0.8" />
+    <xacro:macro name="cylinder_inertia" params="mass length radius">
+        <inertial>
+            <mass value="${mass}" />
+            <inertia ixx="${(mass/12)*(3*radius*radius + length*length)}"
+                     iyy="${(mass/12)*(3*radius*radius + length*length)}"
+                     iyz="0.0" ixy="0.0" ixz="0.0"
+                     izz="${(mass/2)*(radius*radius)}" />
+        </inertial>
+    </xacro:macro>
+    <xacro:macro name="cuboid_inertia" params="mass length breadth height">
+        <inertial>
+            <mass value="${mass}" />
+            <inertia ixx="${(mass/12)*(breadth*breadth + height*height)}"
+                     iyy="${(mass/12)*(height*height + length*length)}"
+                     iyz="0.0" ixy="0.0" ixz="0.0"
+                     izz="${(mass/12)*(breadth*breadth + length*length)}" />
+        </inertial>
+    </xacro:macro>
+    <xacro:macro name="sphere_inertia" params="mass radius">
+        <inertial>
+            <mass value="${mass}" />
+            <inertia ixx="${(mass*0.4)*(radius*radius)}"
+                     iyy="${(mass*0.4)*(radius*radius)}"
+                     iyz="0.0" ixy="0.0" ixz="0.0"
+                     izz="${(mass*0.4)*(radius*radius)}" />
+        </inertial>
+    </xacro:macro>
     <material name="black">
         <color rgba="0.0 0.0 0.0 1.0"/>
@@ -23,5 +57,5 @@
         <visual>
             <geometry>
-                <box size='0.0 0.0 0.0'/>
+                <box size='0.01 0.01 0.01'/>
             </geometry>
             <origin xyz='0.0 0.0 0.0' rpy='0.0 0.0 0.0' />
@@ -39,6 +73,13 @@
             </geometry>
             <origin xyz='0.0 0.0 0.0' rpy='0.0 0.0 0.0' />
-        <material name="black"/>
-        </visual>
+            <material name="black"/>
+        </visual>
+        <collision>
+            <geometry>
+                <box size='${base_length} ${base_length} 0.1'/>
+            </geometry>
+            <origin xyz='0.0 0.0 0.0' rpy='0.0 0.0 0.0' />
+        </collision>
+        <xacro:cuboid_inertia mass="${base_mass}" length="${base_length}" breadth="${base_length}" height="0.1"/>
     </link>
     <joint name="joint1" type="revolute">
@@ -55,5 +96,5 @@
             </geometry>
             <origin xyz='0.0 0.0 ${link1_length/2}' rpy='0.0 0.0 0.0' />
-        <material name="grey"/>
+            <material name="grey"/>
         </visual>
         <visual>
@@ -62,6 +103,13 @@
             </geometry>
             <origin xyz='0.0 0.0 ${link1_length}' rpy='1.57 0.0 0.0' />
-        <material name="grey"/>
-        </visual>
+            <material name="grey"/>
+        </visual>
+        <collision>
+            <geometry>
+                <cylinder length="${link1_length*csf}" radius="${link1_radius}"/>
+            </geometry>
+            <origin xyz='0.0 0.0 ${(link1_length/2)*csf}' rpy='0.0 0.0 0.0' />
+        </collision>
+        <xacro:cylinder_inertia mass="${link1_mass}" radius="${link1_radius}" length="${link1_length}" />
     </link>
     <joint name="joint2" type="revolute">
@@ -78,5 +126,5 @@
             </geometry>
             <origin xyz='${link2_length/2} 0.0 0.0' rpy='0.0 1.57 0.0' />
-        <material name="light_grey"/>
+            <material name="light_grey"/>
         </visual>
         <visual>
@@ -85,6 +133,13 @@
             </geometry>
             <origin xyz='${link2_length} 0.0 0.0' rpy='0.0 0.0 0.0' />
-        <material name="light_grey"/>
-        </visual>
+            <material name="light_grey"/>
+        </visual>
+        <collision>
+            <geometry>
+                <cylinder length="${link2_length*csf}" radius="${link2_radius}"/>
+            </geometry>
+            <origin xyz='${(link2_length/2)*csf} 0.0 0.0' rpy='0.0 1.57 0.0' />
+        </collision>
+        <xacro:cylinder_inertia mass="${link2_mass}" radius="${link2_radius}" length="${link2_length}" />
     </link>
     <joint name="joint3" type="revolute">
@@ -93,5 +148,5 @@
         <origin xyz="${link2_length} 0.0 0.0" rpy="0 0 0.0" />
         <axis xyz="0 0 1" />
-        <limit effort="30" velocity="1.0" lower="-2.13" upper="2.13"/>
+        <limit effort="30" velocity="1.0" lower="-2.00" upper="2.00"/>
     </joint>
     <link name="link3">
@@ -101,6 +156,13 @@
             </geometry>
             <origin xyz='${link3_length/2} 0.0 0.0' rpy='0.0 1.57 0.0' />
-        <material name="lighter_grey"/>
-        </visual>
+            <material name="lighter_grey"/>
+        </visual>
+        <collision>
+            <geometry>
+                <cylinder length="${link3_length*csf}" radius="${link3_radius}"/>
+            </geometry>
+            <origin xyz='${(link3_length/2)*csf} 0.0 0.0' rpy='0.0 1.57 0.0' />
+        </collision>
+        <xacro:cylinder_inertia mass="${link3_mass}" radius="${link3_radius}" length="${link3_length}" />
     </link>
     <joint name="joint_ee" type="fixed">
@@ -116,6 +178,46 @@
             </geometry>
             <origin xyz='0.0 0.0 0.0' rpy='0.0 0.0 0.0' />
-        <material name="lighter_grey"/>
-        </visual>
-    </link>
+            <material name="lighter_grey"/>
+        </visual>
+        <collision>
+            <geometry>
+                <sphere radius="0.03"/>
+            </geometry>
+            <origin xyz='0.0 0.0 0.0' rpy='0.0 0.0 0.0' />
+        </collision>
+        <xacro:sphere_inertia mass="${ee_mass}" radius="0.03" />
+    </link>
+    <transmission name="joint1_trans">
+        <type>transmission_interface/SimpleTransmission</type>
+        <actuator name="$joint1_motor">
+            <mechanicalReduction>1</mechanicalReduction>
+        </actuator>
+        <joint name="joint1">
+            <hardwareInterface>hardware_interface/EffortJointInterface</hardwareInterface>
+        </joint>
+    </transmission>
+    <transmission name="joint2_trans">
+        <type>transmission_interface/SimpleTransmission</type>
+        <actuator name="$joint2_motor">
+            <mechanicalReduction>1</mechanicalReduction>
+        </actuator>
+        <joint name="joint2">
+            <hardwareInterface>hardware_interface/EffortJointInterface</hardwareInterface>
+        </joint>
+    </transmission>
+    <transmission name="joint3_trans">
+        <type>transmission_interface/SimpleTransmission</type>
+        <actuator name="$joint3_motor">
+            <mechanicalReduction>1</mechanicalReduction>
+        </actuator>
+        <joint name="joint3">
+            <hardwareInterface>hardware_interface/EffortJointInterface</hardwareInterface>
+        </joint>
+    </transmission>
+    <!-- plugin for gazebo -->
+    <gazebo>
+        <plugin name="gazebo_ros_control" filename="libgazebo_ros_control.so">
+            <robotNamespace>/</robotNamespace>
+        </plugin>
+    </gazebo>
 </robot>

Commit message: [msm] Found some promising pid value for joint 3

File: my_simple_manipulator/ros/config/my_robot.xacro (robot description, xacro)
@@ -10,7 +10,7 @@
     <xacro:property name="link1_mass" value="1.0" />
     <xacro:property name="link2_mass" value="0.6" />
-    <xacro:property name="link3_mass" value="0.4" />
+    <xacro:property name="link3_mass" value="0.2" />
     <xacro:property name="base_mass" value="10.0" />
-    <xacro:property name="ee_mass" value="0.2" />
+    <xacro:property name="ee_mass" value="0.02" />
     <!-- collision_shortening_factor -->
     <xacro:property name="csf" value="0.8" />
@@ -88,5 +88,5 @@
         <origin xyz="0 0 0.05" rpy="0 0 0.0" />
         <axis xyz="0 0 1" />
-        <limit effort="30" velocity="1.0" lower="-3.13" upper="3.13"/>
+        <limit effort="300" velocity="1.0" lower="-3.13" upper="3.13"/>
     </joint>
     <link name="link1">
@@ -118,5 +118,5 @@
         <origin xyz="0 0 ${link1_length}" rpy="1.57 -1.57 0.0" />
         <axis xyz="0 0 1" />
-        <limit effort="30" velocity="1.0" lower="-2.13" upper="2.13"/>
+        <limit effort="300" velocity="1.0" lower="-2.13" upper="2.13"/>
     </joint>
     <link name="link2">
@@ -148,5 +148,5 @@
         <origin xyz="${link2_length} 0.0 0.0" rpy="0 0 0.0" />
         <axis xyz="0 0 1" />
-        <limit effort="30" velocity="1.0" lower="-2.00" upper="2.00"/>
+        <limit effort="300" velocity="1.0" lower="-2.00" upper="2.00"/>
     </joint>
     <link name="link3">
@@ -191,4 +191,5 @@
         <type>transmission_interface/SimpleTransmission</type>
         <actuator name="$joint1_motor">
+            <hardwareInterface>hardware_interface/EffortJointInterface</hardwareInterface>
             <mechanicalReduction>1</mechanicalReduction>
         </actuator>
@@ -200,4 +201,5 @@
         <type>transmission_interface/SimpleTransmission</type>
         <actuator name="$joint2_motor">
+            <hardwareInterface>hardware_interface/EffortJointInterface</hardwareInterface>
             <mechanicalReduction>1</mechanicalReduction>
         </actuator>
@@ -209,4 +211,5 @@
         <type>transmission_interface/SimpleTransmission</type>
         <actuator name="$joint3_motor">
+            <hardwareInterface>hardware_interface/EffortJointInterface</hardwareInterface>
             <mechanicalReduction>1</mechanicalReduction>
         </actuator>

Commit message: [msm] Found stable pid values for all joints (more or less)

File: my_simple_manipulator/ros/config/my_robot.xacro (robot description, xacro)
@@ -10,7 +10,7 @@
     <xacro:property name="link1_mass" value="1.0" />
     <xacro:property name="link2_mass" value="0.6" />
-    <xacro:property name="link3_mass" value="0.2" />
+    <xacro:property name="link3_mass" value="0.4" />
     <xacro:property name="base_mass" value="10.0" />
-    <xacro:property name="ee_mass" value="0.02" />
+    <xacro:property name="ee_mass" value="0.2" />
     <!-- collision_shortening_factor -->
     <xacro:property name="csf" value="0.8" />
@@ -88,5 +88,5 @@
         <origin xyz="0 0 0.05" rpy="0 0 0.0" />
         <axis xyz="0 0 1" />
-        <limit effort="300" velocity="1.0" lower="-3.13" upper="3.13"/>
+        <limit effort="100" velocity="1.0" lower="-3.13" upper="3.13"/>
     </joint>
     <link name="link1">
@@ -118,5 +118,5 @@
         <origin xyz="0 0 ${link1_length}" rpy="1.57 -1.57 0.0" />
         <axis xyz="0 0 1" />
-        <limit effort="300" velocity="1.0" lower="-2.13" upper="2.13"/>
+        <limit effort="100" velocity="1.0" lower="-2.13" upper="2.13"/>
     </joint>
     <link name="link2">
@@ -148,5 +148,5 @@
         <origin xyz="${link2_length} 0.0 0.0" rpy="0 0 0.0" />
         <axis xyz="0 0 1" />
-        <limit effort="300" velocity="1.0" lower="-2.00" upper="2.00"/>
+        <limit effort="100" velocity="1.0" lower="-2.00" upper="2.00"/>
     </joint>
     <link name="link3">
