Commit message: [MSMB] Added laser to mobile base

File: my_simple_mobile_base/ros/description/my_robot.xacro (robot description, xacro)
@@ -1,4 +1,5 @@
 <?xml version="1.0"?>
 <robot xmlns:xacro="http://www.ros.org/wiki/xacro" name="my_simple_mobile_base">
+    <xacro:include filename="$(find my_simple_mobile_base)/ros/description/laser.xacro" />
     <!-- <xacro:property name="base_length" value="0.5" /> -->
     <xacro:property name="base_mass" value="30.0" />
@@ -121,4 +122,8 @@
         <origin xyz="0.2 -0.1 -0.025" rpy="0 0 0.0" />
     </xacro:wheel>
+    <xacro:laser name="laser" parent="base_link" ros_topic="scan"
+                  update_rate="20" min_angle="-3.14" max_angle="3.14">
+        <origin xyz='0.0 0.0 0.05' rpy='0 0 0'/>
+    </xacro:laser>
     <gazebo>
         <plugin name="object_controller" filename="libgazebo_ros_planar_move.so">
